File: VCRDrums/Clap.kicad_sch (KiCad schematic)
At the start: 93 parts, among them Q701 BC847, Q702 BC857, Q703 BC847, Q704 BC847, Q705 BC847, Q706 BC856, Q707 BC856, Q708 BC857, U701 LM13700, U702 LM339, U704 TL074

Commit message: clave VCA math
Changed lines of the file:
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@@
 	)
 	(global_label "CLAP_MONO"
-		(shape input)
+		(shape output)
 		(at 355.092 101.092 0)
 		(fields_autoplaced yes)

Commit message: mcu skeleton
Parts:
- C714: renamed from C723; footprint (none) -> Capacitor_SMD:C_0805_2012Metric
- Q701, Q703, Q704: footprint PCM_4ms_Package_SOT:SOT-23 -> Package_TO_SOT_SMD:SOT-23
- Q706: renamed from Q705; footprint PCM_4ms_Package_SOT:SOT-23 -> Package_TO_SOT_SMD:SOT-23
- Q707: renamed from Q706; footprint PCM_4ms_Package_SOT:SOT-23 -> Package_TO_SOT_SMD:SOT-23
- Q708: renamed from Q707; footprint PCM_4ms_Package_SOT:SOT-23 -> Package_TO_SOT_SMD:SOT-23
- R701, R702, R703, R704, R705, R706, R707, R708, R709, R710, R711, R712, R713, R714, R715, R716, R717: footprint PCM_Resistor_SMD_AKL:R_0805_2012Metric -> Resistor_SMD:R_0805_2012Metric
- R718: renamed from R752; footprint PCM_Resistor_SMD_AKL:R_0805_2012Metric -> Resistor_SMD:R_0805_2012Metric
- R719: renamed from R753; footprint PCM_Resistor_SMD_AKL:R_0805_2012Metric -> Resistor_SMD:R_0805_2012Metric
- R720: renamed from R718; footprint PCM_Resistor_SMD_AKL:R_0805_2012Metric -> Resistor_SMD:R_0805_2012Metric
- R721: renamed from R749; footprint PCM_Resistor_SMD_AKL:R_0805_2012Metric -> Resistor_SMD:R_0805_2012Metric
- R722: renamed from R719; footprint PCM_Resistor_SMD_AKL:R_0805_2012Metric -> Resistor_SMD:R_0805_2012Metric
- R723: renamed from R720; footprint PCM_Resistor_SMD_AKL:R_0805_2012Metric -> Resistor_SMD:R_0805_2012Metric
- R724: renamed from R754; footprint PCM_Resistor_SMD_AKL:R_0805_2012Metric -> Resistor_SMD:R_0805_2012Metric
- R725: renamed from R721; footprint PCM_Resistor_SMD_AKL:R_0805_2012Metric -> Resistor_SMD:R_0805_2012Metric
- R726: renamed from R722; footprint PCM_Resistor_SMD_AKL:R_0805_2012Metric -> Resistor_SMD:R_0805_2012Metric
- R727: renamed from R723; footprint PCM_Resistor_SMD_AKL:R_0805_2012Metric -> Resistor_SMD:R_0805_2012Metric
- R728: renamed from R748; footprint PCM_Resistor_SMD_AKL:R_0805_2012Metric -> Resistor_SMD:R_0805_2012Metric
- R729: renamed from R724; footprint PCM_Resistor_SMD_AKL:R_0805_2012Metric -> Resistor_SMD:R_0805_2012Metric
- R730: renamed from R725; footprint PCM_Resistor_SMD_AKL:R_0805_2012Metric -> Resistor_SMD:R_0805_2012Metric
- R731: renamed from R750; footprint PCM_Resistor_SMD_AKL:R_0805_2012Metric -> Resistor_SMD:R_0805_2012Metric
- R732: renamed from R726; footprint PCM_Resistor_SMD_AKL:R_0805_2012Metric -> Resistor_SMD:R_0805_2012Metric
- R733: renamed from R727; footprint PCM_Resistor_SMD_AKL:R_0805_2012Metric -> Resistor_SMD:R_0805_2012Metric
- R734: renamed from R728; footprint PCM_Resistor_SMD_AKL:R_0805_2012Metric -> Resistor_SMD:R_0805_2012Metric
- R735: renamed from R746; footprint PCM_Resistor_SMD_AKL:R_0805_2012Metric -> Resistor_SMD:R_0805_2012Metric
- R736: renamed from R729; footprint PCM_Resistor_SMD_AKL:R_0805_2012Metric -> Resistor_SMD:R_0805_2012Metric
- R737: renamed from R747; footprint PCM_Resistor_SMD_AKL:R_0805_2012Metric -> Resistor_SMD:R_0805_2012Metric
- R738: renamed from R745; footprint PCM_Resistor_SMD_AKL:R_0805_2012Metric -> Resistor_SMD:R_0805_2012Metric
- R739: renamed from R730; footprint PCM_Resistor_SMD_AKL:R_0805_2012Metric -> Resistor_SMD:R_0805_2012Metric
- R740: renamed from R731; footprint PCM_Resistor_SMD_AKL:R_0805_2012Metric -> Resistor_SMD:R_0805_2012Metric
- R741: renamed from R751; footprint PCM_Resistor_SMD_AKL:R_0805_2012Metric -> Resistor_SMD:R_0805_2012Metric
- R742: renamed from R732; footprint PCM_Resistor_SMD_AKL:R_0805_2012Metric -> Resistor_SMD:R_0805_2012Metric
- R743: renamed from R734; footprint PCM_Resistor_SMD_AKL:R_0805_2012Metric -> Resistor_SMD:R_0805_2012Metric
- R744: renamed from R735; footprint PCM_Resistor_SMD_AKL:R_0805_2012Metric -> Resistor_SMD:R_0805_2012Metric
- R745: renamed from R733; footprint PCM_Resistor_SMD_AKL:R_0805_2012Metric -> Resistor_SMD:R_0805_2012Metric
- R746: renamed from R736; footprint PCM_Resistor_SMD_AKL:R_0805_2012Metric -> Resistor_SMD:R_0805_2012Metric
- R747: renamed from R737; footprint PCM_Resistor_SMD_AKL:R_0805_2012Metric -> Resistor_SMD:R_0805_2012Metric
- R748: renamed from R738; footprint PCM_Resistor_SMD_AKL:R_0805_2012Metric -> Resistor_SMD:R_0805_2012Metric
- R749: renamed from R739; footprint PCM_Resistor_SMD_AKL:R_0805_2012Metric -> Resistor_SMD:R_0805_2012Metric
- R750: renamed from R740; footprint PCM_Resistor_SMD_AKL:R_0805_2012Metric -> Resistor_SMD:R_0805_2012Metric
- R751: renamed from R741; footprint PCM_Resistor_SMD_AKL:R_0805_2012Metric -> Resistor_SMD:R_0805_2012Metric
- R752: renamed from R742; footprint PCM_Resistor_SMD_AKL:R_0805_2012Metric -> Resistor_SMD:R_0805_2012Metric
- R753: renamed from R743; footprint PCM_Resistor_SMD_AKL:R_0805_2012Metric -> Resistor_SMD:R_0805_2012Metric
- R754: renamed from R744; footprint PCM_Resistor_SMD_AKL:R_0805_2012Metric -> Resistor_SMD:R_0805_2012Metric
- RV701: footprint Potentiometer_THT:Potentiometer_Piher_PT-6-V_Vertical -> Potentiometer_THT:Potentiometer_Bourns_3296W_Vertical
- U701: footprint Package_DIP:DIP-16_W7.62mm -> Package_SO:SOIC-16_3.9x9.9mm_P1.27mm
- U702: footprint PCM_Package_SO_AKL:SOIC-14_3.9x8.7mm_P1.27mm -> Package_SO:SOIC-14_3.9x8.7mm_P1.27mm
- U703: renamed from U704; footprint (none) -> Package_SO:SOIC-14_3.9x8.7mm_P1.27mm
- renumbered C722 to C701, C719 to C702, C718 to C703, C720 to C704, C721 to C705, C701 to C706, C702 to C707, C724 to C708, C704 to C709, C705 to C710, C706 to C711, C707 to C712, C708 to C713, C709 to C715, C710 to C716, C711 to C717, C712 to C718, C713 to C719, C714 to C720, C715 to C721, C716 to C722, C703 to C723, Q708 to Q705
