File: VCRDrums/Clave.kicad_sch (KiCad schematic)
At the start: 66 parts, among them Q801 BC847, Q802 BC856, Q803 BC847, Q804 BC847, Q805 MPF4393, Q806 BC857, U801 LM13700, U803 TL074

Commit message: mcu skeleton
Parts:
- C804: renamed from C813; footprint (none) -> Capacitor_SMD:C_0805_2012Metric
- C805: renamed from C814; footprint (none) -> Capacitor_SMD:C_0805_2012Metric
- C810: renamed from C815; footprint (none) -> Capacitor_SMD:C_0805_2012Metric
- Q801, Q802, Q803: footprint PCM_4ms_Package_SOT:SOT-23 -> Package_TO_SOT_SMD:SOT-23
- Q805: renamed from Q804; footprint PCM_4ms_Package_SOT:SOT-23 -> Package_TO_SOT_SMD:SOT-23
- R801, R802, R803, R804, R805, R806, R807, R808, R809, R810, R811, R812, R813: footprint PCM_Resistor_SMD_AKL:R_0805_2012Metric -> Resistor_SMD:R_0805_2012Metric
- R814: renamed from R827; footprint (none) -> Resistor_SMD:R_0805_2012Metric
- R815: renamed from R828; footprint (none) -> Resistor_SMD:R_0805_2012Metric
- R816: renamed from R814; footprint PCM_Resistor_SMD_AKL:R_0805_2012Metric -> Resistor_SMD:R_0805_2012Metric
- R817: renamed from R829; footprint (none) -> Resistor_SMD:R_0805_2012Metric
- R818: renamed from R830; footprint (none) -> Resistor_SMD:R_0805_2012Metric
- R819: renamed from R815; footprint PCM_Resistor_SMD_AKL:R_0805_2012Metric -> Resistor_SMD:R_0805_2012Metric
- R820: renamed from R831; footprint (none) -> Resistor_SMD:R_0805_2012Metric
- R821: renamed from R816; footprint PCM_Resistor_SMD_AKL:R_0805_2012Metric -> Resistor_SMD:R_0805_2012Metric
- R822: renamed from R817; footprint PCM_Resistor_SMD_AKL:R_0805_2012Metric -> Resistor_SMD:R_0805_2012Metric
- R823: renamed from R832; footprint (none) -> Resistor_SMD:R_0805_2012Metric
- R824: renamed from R818; footprint PCM_Resistor_SMD_AKL:R_0805_2012Metric -> Resistor_SMD:R_0805_2012Metric
- R825: renamed from R819; footprint PCM_Resistor_SMD_AKL:R_0805_2012Metric -> Resistor_SMD:R_0805_2012Metric
- R826: renamed from R833; footprint (none) -> Resistor_SMD:R_0805_2012Metric
- R827: renamed from R834; footprint (none) -> Resistor_SMD:R_0805_2012Metric
- R828: renamed from R835; footprint (none) -> Resistor_SMD:R_0805_2012Metric
- R829: renamed from R820; footprint PCM_Resistor_SMD_AKL:R_0805_2012Metric -> Resistor_SMD:R_0805_2012Metric
- R830: renamed from R836; footprint (none) -> Resistor_SMD:R_0805_2012Metric
- R831: renamed from R821; footprint PCM_Resistor_SMD_AKL:R_0805_2012Metric -> Resistor_SMD:R_0805_2012Metric
- R832: renamed from R822; footprint PCM_Resistor_SMD_AKL:R_0805_2012Metric -> Resistor_SMD:R_0805_2012Metric
- R833: renamed from R823; footprint PCM_Resistor_SMD_AKL:R_0805_2012Metric -> Resistor_SMD:R_0805_2012Metric
- R834: renamed from R837; footprint (none) -> Resistor_SMD:R_0805_2012Metric
- R835: renamed from R838; footprint (none) -> Resistor_SMD:R_0805_2012Metric
- R836: renamed from R824; footprint PCM_Resistor_SMD_AKL:R_0805_2012Metric -> Resistor_SMD:R_0805_2012Metric
- R837: renamed from R825; footprint PCM_Resistor_SMD_AKL:R_0805_2012Metric -> Resistor_SMD:R_0805_2012Metric
- R838: renamed from R826; footprint PCM_Resistor_SMD_AKL:R_0805_2012Metric -> Resistor_SMD:R_0805_2012Metric
- R839: footprint (none) -> Resistor_SMD:R_0805_2012Metric
- U801: renamed from U803; footprint (none) -> Package_SO:SOIC-14_3.9x8.7mm_P1.27mm
- U802: renamed from U801; footprint (none) -> Package_SO:SOIC-16_3.9x9.9mm_P1.27mm
- renumbered C811 to C802, C812 to C803, C802 to C806, C803 to C807, C804 to C808, C805 to C809, C806 to C811, C807 to C812, C808 to C813, C809 to C814, C810 to C815, Q806 to Q804, Q805 to Q806
