File: VCRDrums/Noise.kicad_sch (KiCad schematic)
At the start: 37 parts, among them Q401 BC847, Q402 BC847, U401 40106, U402 TL072

Commit message: mcu skeleton
Parts:
- C408: renamed from C412; footprint (none) -> Capacitor_SMD:C_0805_2012Metric
- C411: renamed from C410; footprint (none) -> Capacitor_SMD:C_0805_2012Metric
- C412: renamed from C413; footprint (none) -> Capacitor_SMD:C_0805_2012Metric
- C413: renamed from C414; footprint (none) -> Capacitor_SMD:C_0805_2012Metric
- Q401, Q402: footprint PCM_4ms_Package_SOT:SOT-23 -> Package_TO_SOT_SMD:SOT-23
- R401, R402, R403, R404, R405, R406, R407, R408, R409, R410, R411, R412, R413, R414, R415, R416, R417, R418, R419: footprint PCM_Resistor_SMD_AKL:R_0805_2012Metric -> Resistor_SMD:R_0805_2012Metric
- U401: footprint PCM_Package_SO_AKL:SOIC-14_3.9x8.7mm_P1.27mm -> Package_SO:SOIC-14_3.9x8.7mm_P1.27mm
- renumbered C408 to C409, C409 to C410, C411 to C414
