File: VCRDrums/Kick.kicad_sch (KiCad schematic)
At the start: 170 parts, among them Q201 BC847, Q202 BC847, Q203 BC847, Q204 BC857, Q205 BC857, Q206 BC857, Q207 BC847, Q208 BC857, Q209 BC847, Q210 BC847, Q211 BC857, Q212 BC857, U201 TL074, U202 LM13700, U203 LM13700, U204 TL074, U205 LM13700, U206 TL074, U207 LM13700, U208 TL074

Commit message: fixed ugly commit history
Changed lines of the file:
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@@
 	(wire
 		(pts
-			(xy 201.676 90.932) (xy 205.994 90.932)
+			(xy 201.676 90.932) (xy 214.63 90.932)
 		)
 		(stroke
@@
 	(wire
 		(pts
-			(xy 215.9 90.932) (xy 210.82 90.932)
+			(xy 215.9 90.932) (xy 215.646 90.932)
 		)
 		(stroke
@@
 	(wire
 		(pts
-			(xy 206.756 352.044) (xy 206.756 351.028)
+			(xy 211.836 352.044) (xy 211.836 354.076)
 		)
 		(stroke
@@
 	(wire
 		(pts
-			(xy 210.566 349.25) (xy 210.566 346.964)
-		)
-		(stroke
-			(width 0)
-			(type default)
-		)
-	)
-	(wire
-		(pts
 			(xy 227.076 349.504) (xy 229.616 349.504)
 		)
@@
 	(wire
 		(pts
-			(xy 197.612 352.044) (xy 201.93 352.044)
+			(xy 197.612 352.044) (xy 210.566 352.044)
 		)
 		(stroke
@@
 	(wire
 		(pts
-			(xy 210.82 90.932) (xy 210.82 89.916)
+			(xy 215.646 90.932) (xy 215.646 92.456)
 		)
 		(stroke
@@
 	(wire
 		(pts
-			(xy 211.836 352.044) (xy 206.756 352.044)
-		)
-		(stroke
-			(width 0)
-			(type default)
-		)
-	)
-	(wire
-		(pts
 			(xy 210.82 456.184) (xy 219.202 456.184)
 		)
@@
 	(wire
 		(pts
-			(xy 214.63 88.138) (xy 214.63 85.852)
+			(xy 214.63 85.852) (xy 214.63 90.932)
 		)
 		(stroke
@@
 	(wire
 		(pts
-			(xy 202.946 89.916) (xy 202.946 85.852)
+			(xy 202.946 92.456) (xy 202.946 85.852)
 		)
 		(stroke
@@
 	(wire
 		(pts
-			(xy 210.82 89.916) (xy 202.946 89.916)
+			(xy 215.646 92.456) (xy 202.946 92.456)
 		)
 		(stroke
@@
 	(wire
 		(pts
-			(xy 206.756 351.028) (xy 198.882 351.028)
+			(xy 211.836 354.076) (xy 198.882 354.076)
 		)
 		(stroke
@@
 	(wire
 		(pts
-			(xy 201.93 349.25) (xy 210.566 349.25)
-		)
-		(stroke
-			(width 0)
-			(type default)
-		)
-	)
-	(wire
-		(pts
 			(xy 216.662 131.572) (xy 216.662 113.792)
 		)
@@
 	(wire
 		(pts
-			(xy 205.994 90.932) (xy 205.994 88.138)
-		)
-		(stroke
-			(width 0)
-			(type default)
-		)
-	)
-	(wire
-		(pts
 			(xy 183.642 139.446) (xy 183.896 139.446)
 		)
@@
 	(wire
 		(pts
-			(xy 205.994 88.138) (xy 214.63 88.138)
-		)
-		(stroke
-			(width 0)
-			(type default)
-		)
-	)
-	(wire
-		(pts
 			(xy 103.124 75.184) (xy 103.124 76.708)
 		)
@@
 	(wire
 		(pts
-			(xy 198.882 351.028) (xy 198.882 346.964)
+			(xy 198.882 354.076) (xy 198.882 346.964)
 		)
 		(stroke
@@
 	(wire
 		(pts
-			(xy 201.93 352.044) (xy 201.93 349.25)
+			(xy 210.566 346.964) (xy 210.566 352.044)
 		)
 		(stroke

Commit message: mcu skeleton
Parts:
- C201: renamed from C220; footprint (none) -> Capacitor_SMD:C_0805_2012Metric
- C202: renamed from C221; footprint (none) -> Capacitor_SMD:C_0805_2012Metric
- C203: renamed from C208; footprint (none) -> Capacitor_SMD:C_0805_2012Metric
- C204: renamed from C209; footprint (none) -> Capacitor_SMD:C_0805_2012Metric
- C205: renamed from C222; footprint (none) -> Capacitor_SMD:C_0805_2012Metric
- C206: renamed from C223; footprint (none) -> Capacitor_SMD:C_0805_2012Metric
- C207: renamed from C224; footprint (none) -> Capacitor_SMD:C_0805_2012Metric
- C208: renamed from C206; footprint (none) -> Capacitor_SMD:C_0805_2012Metric
- C209: renamed from C201; footprint (none) -> Capacitor_SMD:C_0805_2012Metric
- C210: renamed from C207; footprint (none) -> Capacitor_SMD:C_0805_2012Metric
- C211: renamed from C225; footprint (none) -> Capacitor_SMD:C_0805_2012Metric
- C212: renamed from C226; footprint (none) -> Capacitor_SMD:C_0805_2012Metric
- C213: renamed from C211; footprint (none) -> Capacitor_SMD:C_0805_2012Metric
- C214: renamed from C212; footprint (none) -> Capacitor_SMD:C_0805_2012Metric
- C215: renamed from C227; footprint (none) -> Capacitor_SMD:C_0805_2012Metric
- C216: renamed from C228; footprint (none) -> Capacitor_SMD:C_0805_2012Metric
- C217: renamed from C214; footprint (none) -> Capacitor_SMD:C_0805_2012Metric
- C218: renamed from C215; footprint (none) -> Capacitor_SMD:C_0805_2012Metric
- C219: renamed from C229; footprint (none) -> Capacitor_SMD:C_0805_2012Metric
- C220: renamed from C210; footprint (none) -> Capacitor_SMD:C_0805_2012Metric
- C221: renamed from C230; footprint (none) -> Capacitor_SMD:C_0805_2012Metric
- C222: renamed from C202; footprint (none) -> Capacitor_SMD:C_0805_2012Metric
- C223: renamed from C231; footprint (none) -> Capacitor_SMD:C_0805_2012Metric
- C224: renamed from C205; footprint (none) -> Capacitor_SMD:C_0805_2012Metric
- C225: renamed from C232; footprint (none) -> Capacitor_SMD:C_0805_2012Metric
- C226: renamed from C216; footprint (none) -> Capacitor_SMD:C_0805_2012Metric
- C227: renamed from C233; footprint (none) -> Capacitor_SMD:C_0805_2012Metric
- C228: renamed from C203; footprint (none) -> Capacitor_SMD:C_0805_2012Metric
- C229: renamed from C234; footprint (none) -> Capacitor_SMD:C_0805_2012Metric
- C230: renamed from C204; footprint (none) -> Capacitor_SMD:C_0805_2012Metric
- C231: renamed from C235; footprint (none) -> Capacitor_SMD:C_0805_2012Metric
- C232: renamed from C213; footprint (none) -> Capacitor_SMD:C_0805_2012Metric
- C233: renamed from C236; footprint (none) -> Capacitor_SMD:C_0805_2012Metric
- C234: renamed from C217; footprint (none) -> Capacitor_SMD:C_0805_2012Metric
- C235: renamed from C237; footprint (none) -> Capacitor_SMD:C_0805_2012Metric
- C236: renamed from C219; footprint (none) -> Capacitor_SMD:C_0805_2012Metric
- C237: renamed from C238; footprint (none) -> Capacitor_SMD:C_0805_2012Metric
- C238: renamed from C218; footprint (none) -> Capacitor_SMD:C_0805_2012Metric
- R201: renamed from R252; footprint (none) -> Resistor_SMD:R_0805_2012Metric
- R202: renamed from R253; footprint (none) -> Resistor_SMD:R_0805_2012Metric
- R203: renamed from R202; footprint (none) -> Resistor_SMD:R_0805_2012Metric
- R204: renamed from R201; footprint (none) -> Resistor_SMD:R_0805_2012Metric
- R205: renamed from R254; footprint (none) -> Resistor_SMD:R_0805_2012Metric
- R206: renamed from R203; footprint (none) -> Resistor_SMD:R_0805_2012Metric
- R207: renamed from R255; footprint (none) -> Resistor_SMD:R_0805_2012Metric
- R208: renamed from R204; footprint (none) -> Resistor_SMD:R_0805_2012Metric
- R209: renamed from R256; footprint (none) -> Resistor_SMD:R_0805_2012Metric
- R210: renamed from R205; footprint (none) -> Resistor_SMD:R_0805_2012Metric
- R211: renamed from R257; footprint (none) -> Resistor_SMD:R_0805_2012Metric
- R212: renamed from R216; footprint (none) -> Resistor_SMD:R_0805_2012Metric
- R213: renamed from R258; footprint (none) -> Resistor_SMD:R_0805_2012Metric
- R214: renamed from R259; footprint (none) -> Resistor_SMD:R_0805_2012Metric
- R215: renamed from R224; footprint (none) -> Resistor_SMD:R_0805_2012Metric
- R216: renamed from R215; footprint (none) -> Resistor_SMD:R_0805_2012Metric
- R217: renamed from R260; footprint (none) -> Resistor_SMD:R_0805_2012Metric
- R218: renamed from R261; footprint (none) -> Resistor_SMD:R_0805_2012Metric
- R219: renamed from R262; footprint (none) -> Resistor_SMD:R_0805_2012Metric
- R220: renamed from R206; footprint (none) -> Resistor_SMD:R_0805_2012Metric
- R221: renamed from R219; footprint (none) -> Resistor_SMD:R_0805_2012Metric
- R222: renamed from R241; footprint (none) -> Resistor_SMD:R_0805_2012Metric
- R223: renamed from R263; footprint (none) -> Resistor_SMD:R_0805_2012Metric
- R224: renamed from R218; footprint (none) -> Resistor_SMD:R_0805_2012Metric
- R225: renamed from R264; footprint (none) -> Resistor_SMD:R_0805_2012Metric
- R226: renamed from R265; footprint (none) -> Resistor_SMD:R_0805_2012Metric
- R227: renamed from R223; footprint (none) -> Resistor_SMD:R_0805_2012Metric
- R228: renamed from R211; footprint (none) -> Resistor_SMD:R_0805_2012Metric
- R229: renamed from R266; footprint (none) -> Resistor_SMD:R_0805_2012Metric
- R230: renamed from R267; footprint (none) -> Resistor_SMD:R_0805_2012Metric
- R231: renamed from R268; footprint (none) -> Resistor_SMD:R_0805_2012Metric
- R232: renamed from R269; footprint (none) -> Resistor_SMD:R_0805_2012Metric
- R233: renamed from R270; footprint (none) -> Resistor_SMD:R_0805_2012Metric
- R234: renamed from R271; footprint (none) -> Resistor_SMD:R_0805_2012Metric
- R235: renamed from R221; footprint (none) -> Resistor_SMD:R_0805_2012Metric
- R236: renamed from R214; footprint (none) -> Resistor_SMD:R_0805_2012Metric
- R237: renamed from R207; footprint (none) -> Resistor_SMD:R_0805_2012Metric
- R238: renamed from R213; footprint (none) -> Resistor_SMD:R_0805_2012Metric
- R239: renamed from R212; footprint (none) -> Resistor_SMD:R_0805_2012Metric
- R240: renamed from R272; footprint (none) -> Resistor_SMD:R_0805_2012Metric
- R241: renamed from R242; footprint (none) -> Resistor_SMD:R_0805_2012Metric
- R242: renamed from R208; footprint (none) -> Resistor_SMD:R_0805_2012Metric
- R243: renamed from R273; footprint (none) -> Resistor_SMD:R_0805_2012Metric
- R244: renamed from R222; footprint (none) -> Resistor_SMD:R_0805_2012Metric
- R245: renamed from R274; footprint (none) -> Resistor_SMD:R_0805_2012Metric
- R246: renamed from R275; footprint (none) -> Resistor_SMD:R_0805_2012Metric
- R247: renamed from R276; footprint (none) -> Resistor_SMD:R_0805_2012Metric
- R248: renamed from R277; footprint (none) -> Resistor_SMD:R_0805_2012Metric
- R249: renamed from R210; footprint (none) -> Resistor_SMD:R_0805_2012Metric
- R250: renamed from R209; footprint (none) -> Resistor_SMD:R_0805_2012Metric
- R251: renamed from R243; footprint (none) -> Resistor_SMD:R_0805_2012Metric
- R252: renamed from R220; footprint (none) -> Resistor_SMD:R_0805_2012Metric
- R253: renamed from R278; footprint (none) -> Resistor_SMD:R_0805_2012Metric
- R254: renamed from R217; footprint (none) -> Resistor_SMD:R_0805_2012Metric
- R255: renamed from R279; footprint (none) -> Resistor_SMD:R_0805_2012Metric
- R256: renamed from R280; footprint (none) -> Resistor_SMD:R_0805_2012Metric
- R257: renamed from R281; footprint (none) -> Resistor_SMD:R_0805_2012Metric
- R258: renamed from R225; footprint (none) -> Resistor_SMD:R_0805_2012Metric
- R259: renamed from R231; footprint (none) -> Resistor_SMD:R_0805_2012Metric
- R260: renamed from R247; footprint (none) -> Resistor_SMD:R_0805_2012Metric
- R261: renamed from R282; footprint (none) -> Resistor_SMD:R_0805_2012Metric
- R262: renamed from R283; footprint (none) -> Resistor_SMD:R_0805_2012Metric
- R263: renamed from R284; footprint (none) -> Resistor_SMD:R_0805_2012Metric
- R264: renamed from R230; footprint (none) -> Resistor_SMD:R_0805_2012Metric
- R265: renamed from R248; footprint (none) -> Resistor_SMD:R_0805_2012Metric
- R266: renamed from R246; footprint (none) -> Resistor_SMD:R_0805_2012Metric
- R267: renamed from R285; footprint (none) -> Resistor_SMD:R_0805_2012Metric
- R268: renamed from R286; footprint (none) -> Resistor_SMD:R_0805_2012Metric
- R269: renamed from R287; footprint (none) -> Resistor_SMD:R_0805_2012Metric
- R270: renamed from R228; footprint (none) -> Resistor_SMD:R_0805_2012Metric
- R271: renamed from R288; footprint (none) -> Resistor_SMD:R_0805_2012Metric
- R272: renamed from R227; footprint (none) -> Resistor_SMD:R_0805_2012Metric
- R273: renamed from R229; footprint (none) -> Resistor_SMD:R_0805_2012Metric
- R274: renamed from R245; footprint (none) -> Resistor_SMD:R_0805_2012Metric
- R275: renamed from R289; footprint (none) -> Resistor_SMD:R_0805_2012Metric
- R276: renamed from R232; footprint (none) -> Resistor_SMD:R_0805_2012Metric
- R277: renamed from R290; footprint (none) -> Resistor_SMD:R_0805_2012Metric
- R278: renamed from R249; footprint (none) -> Resistor_SMD:R_0805_2012Metric
- R279: renamed from R291; footprint (none) -> Resistor_SMD:R_0805_2012Metric
- R280: renamed from R235; footprint (none) -> Resistor_SMD:R_0805_2012Metric
- R281: renamed from R292; footprint (none) -> Resistor_SMD:R_0805_2012Metric
- R282: renamed from R293; footprint (none) -> Resistor_SMD:R_0805_2012Metric
- R283: renamed from R233; footprint (none) -> Resistor_SMD:R_0805_2012Metric
- R284: renamed from R226; footprint (none) -> Resistor_SMD:R_0805_2012Metric
- R285: renamed from R294; footprint (none) -> Resistor_SMD:R_0805_2012Metric
- R286: renamed from R244; footprint (none) -> Resistor_SMD:R_0805_2012Metric
- R287: renamed from R295; footprint (none) -> Resistor_SMD:R_0805_2012Metric
- R288: renamed from R234; footprint (none) -> Resistor_SMD:R_0805_2012Metric
- R289: renamed from R296; footprint (none) -> Resistor_SMD:R_0805_2012Metric
- R290: renamed from R297; footprint (none) -> Resistor_SMD:R_0805_2012Metric
- R291: renamed from R298; footprint (none) -> Resistor_SMD:R_0805_2012Metric
- R292: renamed from R238; footprint (none) -> Resistor_SMD:R_0805_2012Metric
- R293: renamed from R239; footprint (none) -> Resistor_SMD:R_0805_2012Metric
- R294: renamed from R251; footprint (none) -> Resistor_SMD:R_0805_2012Metric
- R295: renamed from R299; footprint (none) -> Resistor_SMD:R_0805_2012Metric
- R296: renamed from R300; footprint (none) -> Resistor_SMD:R_0805_2012Metric
- R297: renamed from R328; footprint (none) -> Resistor_SMD:R_0805_2012Metric
- R298: renamed from R250; footprint (none) -> Resistor_SMD:R_0805_2012Metric
- R299: renamed from R236; footprint (none) -> Resistor_SMD:R_0805_2012Metric
- R300: renamed from R237; footprint (none) -> Resistor_SMD:R_0805_2012Metric
- R301: renamed from R329; footprint (none) -> Resistor_SMD:R_0805_2012Metric
- R302: renamed from R240; footprint (none) -> Resistor_SMD:R_0805_2012Metric
- U201: renamed from U205; footprint (none) -> Package_SO:SOIC-16_3.9x9.9mm_P1.27mm
- U202: footprint (none) -> Package_SO:SOIC-16_3.9x9.9mm_P1.27mm
- U203: renamed from U206; footprint (none) -> Package_SO:SOIC-14_3.9x8.7mm_P1.27mm
- U204: renamed from U201; footprint (none) -> Package_SO:SOIC-14_3.9x8.7mm_P1.27mm
- U205: renamed from U207; footprint (none) -> Package_SO:SOIC-16_3.9x9.9mm_P1.27mm
- U206: renamed from U203; footprint (none) -> Package_SO:SOIC-16_3.9x9.9mm_P1.27mm
- U207: renamed from U208; footprint (none) -> Package_SO:SOIC-14_3.9x8.7mm_P1.27mm
- U208: renamed from U204; footprint (none) -> Package_SO:SOIC-14_3.9x8.7mm_P1.27mm
- renumbered D206 to D201, D201 to D202, D207 to D203, D202 to D204, D208 to D205, D203 to D206, D209 to D207, D210 to D208, D204 to D209, D205 to D210, Q207 to Q201, Q201 to Q202, Q208 to Q203, Q209 to Q205, Q202 to Q206, Q210 to Q207, Q203 to Q208, Q211 to Q209, Q206 to Q210, Q212 to Q211, Q205 to Q212

Commit message: compressor schem and schematic
Parts:
- D201, D202, D203, D204, D205, D206, D207, D208, D209, D210: footprint Diode_THT:D_DO-35_SOD27_P7.62mm_Horizontal -> Diode_SMD:D_SOD-123
Changed lines of the file:
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@@
 			)
 		)
-		(property "Footprint" "Diode_THT:D_DO-35_SOD27_P7.62mm_Horizontal"
+		(property "Footprint" "Diode_SMD:D_SOD-123"
 			(at 323.85 237.236 0)
 			(effects
@@
 			)
 		)
-		(property "Footprint" "Diode_THT:D_DO-35_SOD27_P7.62mm_Horizontal"
+		(property "Footprint" "Diode_SMD:D_SOD-123"
 			(at 202.946 118.872 0)
 			(effects
@@
 			)
 		)
-		(property "Footprint" "Diode_THT:D_DO-35_SOD27_P7.62mm_Horizontal"
+		(property "Footprint" "Diode_SMD:D_SOD-123"
 			(at 319.786 498.348 0)
 			(effects
@@
 			)
 		)
-		(property "Footprint" "Diode_THT:D_DO-35_SOD27_P7.62mm_Horizontal"
+		(property "Footprint" "Diode_SMD:D_SOD-123"
 			(at 319.532 488.696 0)
 			(effects
@@
 			)
 		)
-		(property "Footprint" "Diode_THT:D_DO-35_SOD27_P7.62mm_Horizontal"
+		(property "Footprint" "Diode_SMD:D_SOD-123"
 			(at 323.596 227.584 0)
 			(effects
@@
 			)
 		)
-		(property "Footprint" "Diode_THT:D_DO-35_SOD27_P7.62mm_Horizontal"
+		(property "Footprint" "Diode_SMD:D_SOD-123"
 			(at 165.354 400.558 0)
 			(effects
@@
 			)
 		)
-		(property "Footprint" "Diode_THT:D_DO-35_SOD27_P7.62mm_Horizontal"
+		(property "Footprint" "Diode_SMD:D_SOD-123"
 			(at 198.882 379.984 0)
 			(effects
@@
 			)
 		)
-		(property "Footprint" "Diode_THT:D_DO-35_SOD27_P7.62mm_Horizontal"
+		(property "Footprint" "Diode_SMD:D_SOD-123"
 			(at 169.418 139.446 0)
 			(effects
@@
 			)
 		)
-		(property "Footprint" "Diode_THT:D_DO-35_SOD27_P7.62mm_Horizontal"
+		(property "Footprint" "Diode_SMD:D_SOD-123"
 			(at 110.49 435.102 0)
 			(effects
@@
 			)
 		)
-		(property "Footprint" "Diode_THT:D_DO-35_SOD27_P7.62mm_Horizontal"
+		(property "Footprint" "Diode_SMD:D_SOD-123"
 			(at 114.554 173.99 0)
 			(effects
