File: VCRDrums/Mixer.kicad_sch (KiCad schematic)
At the start: 72 parts, among them U301 LM1972, U302 L7805, U303 L7905, U304 LM1972, U305 LM1972, U306 LM1972, U307 LM1972, U308 LM1972, U309 TL074, U310 TL074, U311 TL074, U312 TL074, U313 LM1972, U314 TL074

Commit message: clave VCA math
Parts:
- added R332, R333: 100k, symbol Device:R_US
Connections:
- net at R309.2, R310.2, R311.2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: now also R333.2
- net at R301.2, R302.1, R303.2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: now also R332.2
- net TOM_L renamed CLAVE_L
- net TOM_MONO renamed CLAVE_MONO
- net TOM_R renamed CLAVE_R
- new net DIGITAL_L: R332.1
- new net DIGITAL_R: R333.1
Other:
- note added: "TODO: stereo audio DAC goes here"
- moved on the sheet: C301, C302, C303, C304, C305, C306, C307, C308, C309, C310, C311, C312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

Commit message: mcu skeleton
Parts:
- C301: renamed from C327; footprint (none) -> Capacitor_SMD:C_0805_2012Metric
- C302: renamed from C328; footprint (none) -> Capacitor_SMD:C_0805_2012Metric
- C303: renamed from C317; footprint (none) -> Capacitor_SMD:C_0805_2012Metric
- C304: renamed from C318; footprint (none) -> Capacitor_SMD:C_0805_2012Metric
- C305: renamed from C319; footprint (none) -> Capacitor_SMD:C_0805_2012Metric
- C306: renamed from C320; footprint (none) -> Capacitor_SMD:C_0805_2012Metric
- C307: renamed from C321; footprint (none) -> Capacitor_SMD:C_0805_2012Metric
- C308: renamed from C322; footprint (none) -> Capacitor_SMD:C_0805_2012Metric
- C309: renamed from C323; footprint (none) -> Capacitor_SMD:C_0805_2012Metric
- C310: renamed from C324; footprint (none) -> Capacitor_SMD:C_0805_2012Metric
- C311: renamed from C305; footprint (none) -> Capacitor_SMD:C_0805_2012Metric
- C312: renamed from C313; footprint (none) -> Capacitor_SMD:C_0805_2012Metric
- C313: renamed from C306; footprint (none) -> Capacitor_SMD:C_0805_2012Metric
- C314: footprint (none) -> Capacitor_SMD:C_0805_2012Metric
- C315: renamed from C325; footprint (none) -> Capacitor_SMD:C_0805_2012Metric
- C316: renamed from C315; footprint (none) -> Capacitor_SMD:C_0805_2012Metric
- C317: renamed from C326; footprint (none) -> Capacitor_SMD:C_0805_2012Metric
- C318: renamed from C316; footprint (none) -> Capacitor_SMD:C_0805_2012Metric
- C319: renamed from C301; footprint (none) -> Capacitor_SMD:C_0805_2012Metric
- C320: renamed from C304; footprint (none) -> Capacitor_SMD:C_0805_2012Metric
- C321: renamed from C302; footprint (none) -> Capacitor_SMD:C_0805_2012Metric
- C322: renamed from C303; footprint (none) -> Capacitor_SMD:C_0805_2012Metric
- C323: renamed from C309; footprint (none) -> Capacitor_SMD:C_0805_2012Metric
- C324: renamed from C310; footprint (none) -> Capacitor_SMD:C_0805_2012Metric
- C325: renamed from C307; footprint (none) -> Capacitor_SMD:C_0805_2012Metric
- C326: renamed from C308; footprint (none) -> Capacitor_SMD:C_0805_2012Metric
- C327: renamed from C311; footprint (none) -> Capacitor_SMD:C_0805_2012Metric
- C328: renamed from C312; footprint (none) -> Capacitor_SMD:C_0805_2012Metric
- R303: renamed from R319; footprint (none) -> Resistor_SMD:R_0805_2012Metric
- R304: renamed from R320; footprint (none) -> Resistor_SMD:R_0805_2012Metric
- R305: renamed from R318; footprint (none) -> Resistor_SMD:R_0805_2012Metric
- R306: renamed from R321; footprint (none) -> Resistor_SMD:R_0805_2012Metric
- R307: renamed from R324; footprint (none) -> Resistor_SMD:R_0805_2012Metric
- R308: renamed from R326; footprint (none) -> Resistor_SMD:R_0805_2012Metric
- R309: renamed from R317; footprint (none) -> Resistor_SMD:R_0805_2012Metric
- R310: renamed from R322; footprint (none) -> Resistor_SMD:R_0805_2012Metric
- R311: renamed from R301; footprint (none) -> Resistor_SMD:R_0805_2012Metric
- R312: renamed from R303; footprint (none) -> Resistor_SMD:R_0805_2012Metric
- R313: renamed from R304; footprint (none) -> Resistor_SMD:R_0805_2012Metric
- R314: renamed from R305; footprint (none) -> Resistor_SMD:R_0805_2012Metric
- R315: renamed from R306; footprint (none) -> Resistor_SMD:R_0805_2012Metric
- R316: renamed from R307; footprint (none) -> Resistor_SMD:R_0805_2012Metric
- R317: renamed from R308; footprint (none) -> Resistor_SMD:R_0805_2012Metric
- R318: renamed from R332; footprint (none) -> Resistor_SMD:R_0805_2012Metric
- R319: renamed from R331; footprint (none) -> Resistor_SMD:R_0805_2012Metric
- R320: renamed from R323; footprint (none) -> Resistor_SMD:R_0805_2012Metric
- R321: renamed from R325; footprint (none) -> Resistor_SMD:R_0805_2012Metric
- R322: renamed from R327; footprint (none) -> Resistor_SMD:R_0805_2012Metric
- R323: renamed from R302; footprint (none) -> Resistor_SMD:R_0805_2012Metric
- R324: renamed from R309; footprint (none) -> Resistor_SMD:R_0805_2012Metric
- R325: renamed from R310; footprint (none) -> Resistor_SMD:R_0805_2012Metric
- R326: renamed from R311; footprint (none) -> Resistor_SMD:R_0805_2012Metric
- R327: renamed from R312; footprint (none) -> Resistor_SMD:R_0805_2012Metric
- R328: renamed from R313; footprint (none) -> Resistor_SMD:R_0805_2012Metric
- R329: renamed from R314; footprint (none) -> Resistor_SMD:R_0805_2012Metric
- R330: renamed from R315; footprint (none) -> Resistor_SMD:R_0805_2012Metric
- R331: renamed from R333; footprint (none) -> Resistor_SMD:R_0805_2012Metric
- R332: renamed from R316; footprint (none) -> Resistor_SMD:R_0805_2012Metric
- R333: renamed from R330; footprint (none) -> Resistor_SMD:R_0805_2012Metric
- RV301: footprint (none) -> Potentiometer_THT:Potentiometer_Alpha_RD902F-40-00D_Dual_Vertical
- U301: renamed from U314; footprint (none) -> Package_SO:SOIC-14_3.9x8.7mm_P1.27mm
- U302: renamed from U309; footprint (none) -> Package_SO:SOIC-14_3.9x8.7mm_P1.27mm
- U303: renamed from U310; footprint (none) -> Package_SO:SOIC-14_3.9x8.7mm_P1.27mm
- U304: renamed from U311; footprint (none) -> Package_SO:SOIC-14_3.9x8.7mm_P1.27mm
- U305: renamed from U312; footprint (none) -> Package_SO:SOIC-14_3.9x8.7mm_P1.27mm
- U310: renamed from U302; footprint (none) -> PCM_4ms_Package_TO:TO-220-3_Vertical
- U311: renamed from U303; footprint (none) -> PCM_4ms_Package_TO:TO-220-3_Vertical
- renumbered U301 to U306, U313 to U308, U308 to U309, U305 to U312, U304 to U313, U306 to U314

Commit message: compressor muxes and balanced out
Parts:
- removed RV301: 100k, Potentiometer_THT:Potentiometer_Alpha_RD902F-40-00D_Dual_Vertical, symbol Device:R_Potentiometer_Dual
- removed U301: TL074, Package_SO:SOIC-14_3.9x8.7mm_P1.27mm, symbol Amplifier_Operational:TL074
- added C329, C330, C331, C332, C333, C334, C335, C336, C342, C345, C346, C347, C348, C349, C350, C351, C352: 100n, Capacitor_SMD:C_0805_2012Metric, symbol Device:C
- added C337, C338, C341: 10u, Capacitor_SMD:C_0805_2012Metric, symbol Device:C
- added C339, C340: 2u2, Capacitor_SMD:C_0805_2012Metric, symbol Device:C
- added C343, C344: 2n2, Capacitor_SMD:C_0805_2012Metric, symbol Device:C
- added JP301: DAC_DEMP, symbol Jumper:SolderJumper_2_Open
- added JP302: DAC_FLT, symbol Jumper:SolderJumper_2_Open
- added R334, R336, R337, R338, R339, R340, R341, R342, R343: 100k, Resistor_SMD:R_0805_2012Metric, symbol Device:R_US
- added R335, R344: 33k, Resistor_SMD:R_0805_2012Metric, symbol Device:R_US
- added R345, R346, R347, R348: 470, Resistor_SMD:R_0805_2012Metric, symbol Device:R_US
- added R349, R350, R351, R352: 10k, Resistor_SMD:R_0805_2012Metric, symbol Device:R_US
- added R353, R354, R355, R356: 47k, symbol Device:R_US
- added R357, R358, R359, R360: 10k, symbol Device:R_US
- added RV301, RV302: 100k, symbol Device:R_Potentiometer_Dual_Separate
- added U301, U315, U316, U317, U320, U321: TMUX4053, Package_SO:TSSOP-16_4.4x5mm_P0.65mm, symbol Analog_Switch:TMUX4053
- added U318, U322: TL074, symbol Amplifier_Operational:TL074
- added U319: PCM5100A, Package_SO:TSSOP-20_4.4x6.5mm_P0.65mm, symbol Audio:PCM5100A
- R303, R304, R305: value 100k -> 10k; footprint Resistor_SMD:R_0805_2012Metric -> (none)
- R306: value 100k -> 470
- R307: value 220R -> 470
- R308, R321, R322: value 220R -> 100k
Connections:
- net +12V: now also C302.1, C330.1, C332.1, C334.1, C346.1, C347.1, C350.1, C351.1, U301.16 (VDD), U315.16 (VDD), U316.16 (VDD), U317.16 (VDD), U318.4 (V+), U320.16 (VDD), U321.16 (VDD), U322.4 (V+); no longer C301.1
- net -12V: now also C301.1, C329.1, C331.1, C333.1, C345.1, C348.1, C349.1, C352.1, U301.7 (VSS), U315.7 (VSS), U316.7 (VSS), U317.7 (VSS), U318.11 (V-), U320.7 (VSS), U321.7 (VSS), U322.11 (V-); no longer C302.1
- net CLAP_L: now also U317.14 (A); no longer R317.1
- net CLAP_R: now also U316.4 (C); no longer R330.1
- net CLAVE_L: now also U317.4 (C); no longer R316.1
- net CLAVE_R: now also U317.15 (B); no longer R329.1
- net CLSDHAT_L: now also U316.15 (B); no longer R314.1
- net CLSDHAT_R: now also U316.14 (A); no longer R327.1
- net DIGITAL_L: now also U318.1, U318.2 (-), U321.15 (B); no longer R318.1
- net DIGITAL_R: now also U318.6 (-), U318.7, U321.14 (A); no longer R331.1
- net GND: now also R305.2, C329.2, C330.2, C331.2, C332.2, C333.2, C334.2, C335.2, C336.2, C337.2, C338.2, C339.2, C341.2, C342.2, C343.2, C344.2, C345.2, C346.2, C347.2, C348.2, C349.2, C350.2, C351.2, C352.2, JP301.1 (A), RV301.2, RV301.5, RV302.3, RV302.6, U301.6 (INH), U301.8 (GND), U315.6 (INH), U315.8 (GND), U316.6 (INH), U316.8 (GND), U317.6 (INH), U317.8 (GND), U318.10 (+), U318.12 (+), U319.12 (SCK), U319.16 (FMT), U319.19 (DGND), U319.3 (CPGND), U319.9 (AGND), U320.6 (INH), U320.8 (GND), U321.6 (INH), U321.8 (GND), U322.10 (+), U322.12 (+); no longer R303.2, R304.2
- net KICK1_L: now also U301.15 (B); no longer R311.1
- net KICK1_R: now also U301.14 (A); no longer R324.1
- net KICK2_L: now also U315.14 (A); no longer R312.1
- net KICK2_R: now also U301.4 (C); no longer R325.1
- net OPENHAT_L: now also U315.4 (C); no longer R313.1
- net OPENHAT_R: now also U315.15 (B); no longer R326.1
- net SNARE_L: now also U320.15 (B); no longer R315.1
- net SNARE_R: now also U320.14 (A); no longer R328.1
- net at R320.2, R322.2: now also R308.2, R309.2, R310.2, R319.2, R321.2, R334.2, R335.1, U318.9 (-)
- net SNARE_L_COMP: now reaches R320.1
- net SNARE_L_COMP: now also U320.2 (B0); no longer R310.2
- net at R305.1: now also JP302.1 (A), U319.11 (FLT); no longer R303.1
- net CLSDHAT_L_COMP: now reaches R319.1
- net CLSDHAT_L_COMP: now also U316.2 (B0); no longer R309.2
- net at R306.1: now also U319.7 (OUTR); no longer R304.1
- net FULL_L: no longer names the net of R323.2, U305.8
- net FULL_L: now also R346.1
- net FULL_R: no longer names the net of R332.2, U305.14
- net FULL_R: now also R345.1
- net OUTPUT_LEFT_N renamed CLAVE_L_COMP
- net CLAVE_L_COMP: now also U317.5 (C0)
- net OUTPUT_LEFT_P: no longer names the net of R307.1
- net OUTPUT_LEFT_P: now also U319.6 (OUTL)
- net OUTPUT_RIGHT_N renamed CLAP_L_COMP
- net CLAP_L_COMP: now also U317.12 (A0)
- net OUTPUT_RIGHT_P renamed KICK1_L_COMP
- net KICK1_L_COMP: now also U301.2 (B0)
- new net: R355.1, R359.2, U322.6 (-), U322.7
- new net: R355.2, R356.1, U322.9 (-)
- new net: R336.2, R337.2, R338.2, R339.2, R340.2, R341.2, R342.2, R343.2, R344.1, U318.13 (-)
- new net: R348.2, R349.1, RV301.4
- new net: R349.2, R350.2, RV302.4
- new net: R353.1, R357.2, U322.1, U322.2 (-)
- new net: RV302.2, U322.3 (+)
- new net: R351.2, R352.2, RV302.1
- new net: RV302.5, U322.5 (+)
- new net: C341.1, C342.1, U319.18 (LDOO)
- new net: R356.2, R360.2, U322.8
- new net: C339.1, U319.5 (VNEG)
- new net: R353.2, R354.1, U322.13 (-)
- new net: R354.2, R358.2, U322.14
- new net: R347.2, R352.1, RV301.1
- new net: C344.1, R307.2, U318.3 (+)
- new net: C340.1, U319.2 (CAPP)
- new net: C340.2, U319.4 (CAPM)
- new net: C343.1, R306.2, U318.5 (+)
- new net +3.3VA: C335.1, C336.1, C337.1, C338.1, JP302.2 (B), R303.1, R304.1, U319.1 (CPVDD), U319.20 (DVDD), U319.8 (AVDD)
- new net BAL_L+: R357.1
- new net BAL_L-: R358.1
- new net BAL_R+: R359.1
- new net BAL_R-: R360.1
- new net CLAP_COMP_MODE: U316.9 (S3), U317.11 (S1)
- new net CLAP_L_CLN: R317.1, U317.13 (A1)
- new net CLAP_R_CLN: R330.1, U316.3 (C1)
- new net CLAP_R_COMP: R342.1, U316.5 (C0)
- new net CLAVE_COMP_MODE: U317.10 (S2), U317.9 (S3)
- new net CLAVE_L_CLN: R316.1, U317.3 (C1)
- new net CLAVE_R_CLN: R329.1, U317.1 (B1)
- new net CLAVE_R_COMP: R341.1, U317.2 (B0)
- new net CLN_L: R346.2, R351.1, RV301.3
- new net CLN_R: R350.1, RV301.6
- new net CLR_R: R345.2
- new net CLSDHAT_COMP_MODE: U316.10 (S2), U316.11 (S1)
- new net CLSDHAT_L_CLN: R314.1, U316.1 (B1)
- new net CLSDHAT_R_CLN: R327.1, U316.13 (A1)
- new net CLSDHAT_R_COMP: R339.1, U316.12 (A0)
- new net COMP_IN_L: R335.2, U318.8
- new net COMP_IN_R: R344.2, U318.14
- new net COMP_OUT_L: R347.1
- new net COMP_OUT_R: R348.1
- new net DAC_UNMUTE: R303.2, U319.17 (XSMT)
- new net DEMP: JP301.2 (B), R304.2, U319.10 (DEMP)
- new net DIGITAL_COMP_MODE: U321.10 (S2), U321.11 (S1)
- new net DIGITAL_L_CLN: R318.1, U321.1 (B1)
- new net DIGITAL_L_COMP: R334.1, U321.2 (B0)
- new net DIGITAL_R_CLN: R331.1, U321.13 (A1)
- new net DIGITAL_R_COMP: R343.1, U321.12 (A0)
- new net I2S_BCK: U319.13 (BCK)
- new net I2S_DIN: U319.14 (DIN)
- new net I2S_LRCK: U319.15 (LRCK)
- new net KICK1_COMP_MODE: U301.10 (S2), U301.11 (S1)
- new net KICK1_L_CLN: R311.1, U301.1 (B1)
- new net KICK1_R_CLN: R324.1, U301.13 (A1)
- new net KICK1_R_COMP: R336.1, U301.12 (A0)
- new net KICK2_COMP_MODE: U301.9 (S3), U315.11 (S1)
- new net KICK2_L_CLN: R312.1, U315.13 (A1)
- new net KICK2_L_COMP: R309.1, U315.12 (A0)
- new net KICK2_R_CLN: R325.1, U301.3 (C1)
- new net KICK2_R_COMP: R337.1, U301.5 (C0)
- new net OPENHAT_COMP_MODE: U315.10 (S2), U315.9 (S3)
- new net OPENHAT_L_CLN: R313.1, U315.3 (C1)
- new net OPENHAT_L_COMP: R310.1, U315.5 (C0)
- new net OPENHAT_R_CLN: R326.1, U315.1 (B1)
- new net OPENHAT_R_COMP: R338.1, U315.2 (B0)
- new net SNARE_COMP_MODE: U320.10 (S2), U320.11 (S1)
- new net SNARE_L_CLN: R315.1, U320.1 (B1)
- new net SNARE_R_CLN: R328.1, U320.13 (A1)
- new net SNARE_R_COMP: R340.1, U320.12 (A0)
- no-connect marks 0 -> 8
Other:
- note added: "RV301 - Compressor wet/dry control (linear) RV302 - Master Volume (audio taper)"
- note removed: "TODO: stereo audio DAC goes here"
- note removed: "Volume control & balanced outputs"
- moved on the sheet: C303, C304, C305, C306, C307, C308, C309, C310, C311, C312, C313, C314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

Commit message: compressor schem and schematic
Parts:
- JP301, JP302: footprint (none) -> Jumper:SolderJumper-2_P1.3mm_Open_RoundedPad1.0x1.5mm
- R303, R304, R305, R353, R354, R355, R356, R357, R358, R359, R360, RV301, RV302, U318, U322: footprint (none) -> Resistor_SMD:R_0805_2012Metric
Connections:
- net +3.3VA: no longer C335.1, C336.1, C337.1, C338.1, U319.1 (CPVDD), U319.20 (DVDD), U319.8 (AVDD)
- new net +3.3VP: C335.1, C336.1, C337.1, C338.1, U319.1 (CPVDD), U319.20 (DVDD), U319.8 (AVDD)
Other:
- moved on the sheet: C331, C332, C349, C350, U316, U321
